File: CurrentVersion/Hardware/EagleCircuit/V2.0.brd (EAGLE design)
At the start: 53 x 45.7 mm, 16 parts

Commit message: New pcb
Parts:
- removed S1: 2P2T, switch:2P2T
- added S3: (no value), switch:M251
- renumbered JP4 to BATT, JP5 to ROUTER
Connections:
- net RX1: now also JP7.2; no longer JP7.11
- net TX1: now also JP7.1; no longer JP7.10
- net VCC: now also S3.1; no longer S1.3.2
- net VCC2: now also S3.2; no longer S1.2.2
Routing:
- net TX1: track 24.8 -> 46.4 mm
- net RX1: track 28.6 -> 49.4 mm
- net VCC: track 21.9 -> 27.3 mm
- net VCC2: track 36.3 -> 37.0 mm
Changed lines of the file:
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@@
 <element name="R2" library="rcl" package="0204/7" value="" x="46.99" y="19.05" rot="R180"/>
 <element name="U$2" library="SparkFun" package="OSHW-LOGO-S" value="OSHW-LOGOS" x="58.42" y="39.37" rot="R90"/>
-<element name="S1" library="switch" package="2P2T" value="2P2T" x="87.63" y="50.8" rot="R270"/>
-<element name="JP4" library="pinhead" package="1X02/90" value="" x="71.12" y="49.53" smashed="yes">
+<element name="BATT" library="pinhead" package="1X02/90" value="" x="71.12" y="49.53" smashed="yes">
 <attribute name="NAME" x="67.945" y="48.26" size="1.27" layer="25" ratio="10" rot="R270" align="top-right"/>
 <attribute name="VALUE" x="75.565" y="45.72" size="1.27" layer="27" rot="R90"/>
 </element>
-<element name="JP5" library="pinhead" package="1X02/90" value="" x="55.88" y="49.53" smashed="yes">
+<element name="ROUTER" library="pinhead" package="1X02/90" value="" x="55.88" y="49.53" smashed="yes">
 <attribute name="NAME" x="60.325" y="48.26" size="1.27" layer="25" ratio="10" rot="R90"/>
 <attribute name="VALUE" x="60.325" y="45.72" size="1.27" layer="27" rot="R90"/>
 </element>
+<element name="S3" library="switch" package="M251" value="" x="87.63" y="49.53" rot="R90"/>
 </elements>
 <signals>
@@
 <wire x1="45.72" y1="21.59" x2="46.99" y2="22.86" width="0.4064" layer="16"/>
 <wire x1="46.99" y1="22.86" x2="46.99" y2="24.13" width="0.4064" layer="16"/>
-<contactref element="JP5" pad="1"/>
+<contactref element="ROUTER" pad="1"/>
 <wire x1="44.45" y1="45.72" x2="44.45" y2="46.99" width="0.4064" layer="16"/>
 <wire x1="44.45" y1="46.99" x2="45.72" y2="48.26" width="0.4064" layer="16"/>
@@
 </signal>
 <signal name="TX1">
-<contactref element="JP7" pad="10"/>
 <contactref element="R1" pad="1"/>
-<wire x1="58.42" y1="16.51" x2="58.42" y2="15.76605" width="0.4064" layer="16"/>
-<wire x1="58.42" y1="15.76605" x2="60.21605" y2="13.97" width="0.4064" layer="16"/>
-<wire x1="60.21605" y1="13.97" x2="66.78395" y2="13.97" width="0.4064" layer="16"/>
-<wire x1="66.78395" y1="13.97" x2="68.58" y2="15.76605" width="0.4064" layer="16"/>
-<wire x1="68.58" y1="15.76605" x2="68.58" y2="22.33395" width="0.4064" layer="16"/>
-<wire x1="68.58" y1="22.33395" x2="66.78395" y2="24.13" width="0.4064" layer="16"/>
-<wire x1="66.78395" y1="24.13" x2="63.5" y2="24.13" width="0.4064" layer="16"/>
+<contactref element="JP7" pad="1"/>
+<wire x1="63.5" y1="46.99" x2="65.74019375" y2="46.99" width="0.4064" layer="16"/>
+<wire x1="65.74019375" y1="46.99" x2="68.58" y2="44.15019375" width="0.4064" layer="16"/>
+<wire x1="68.58" y1="44.15019375" x2="68.58" y2="16.80980625" width="0.4064" layer="16"/>
+<wire x1="68.58" y1="16.80980625" x2="65.74019375" y2="13.97" width="0.4064" layer="16"/>
+<wire x1="65.74019375" y1="13.97" x2="60.21605" y2="13.97" width="0.4064" layer="16"/>
+<wire x1="60.21605" y1="13.97" x2="58.42" y2="15.76605" width="0.4064" layer="16"/>
+<wire x1="58.42" y1="15.76605" x2="58.42" y2="16.51" width="0.4064" layer="16"/>
 </signal>
 <signal name="RX1">
 <contactref element="JP6" pad="4"/>
-<contactref element="JP7" pad="11"/>
-<wire x1="63.5" y1="21.59" x2="66.04" y2="21.59" width="0.4064" layer="16"/>
-<wire x1="66.04" y1="21.59" x2="67.31" y2="20.32" width="0.4064" layer="16"/>
-<wire x1="67.31" y1="20.32" x2="67.31" y2="17.03605" width="0.4064" layer="16"/>
-<wire x1="67.31" y1="17.03605" x2="65.51395" y2="15.24" width="0.4064" layer="16"/>
-<wire x1="65.51395" y1="15.24" x2="62.97395" y2="15.24" width="0.4064" layer="16"/>
+<contactref element="JP7" pad="2"/>
+<wire x1="63.5" y1="44.45" x2="65.51395" y2="44.45" width="0.4064" layer="16"/>
+<wire x1="65.51395" y1="44.45" x2="67.31" y2="42.65395" width="0.4064" layer="16"/>
+<wire x1="67.31" y1="42.65395" x2="67.31" y2="18.30605" width="0.4064" layer="16"/>
+<wire x1="67.31" y1="18.30605" x2="65.51395" y2="16.51" width="0.4064" layer="16"/>
+<wire x1="65.51395" y1="16.51" x2="61.70395" y2="16.51" width="0.4064" layer="16"/>
+<wire x1="61.70395" y1="16.51" x2="60.96" y2="17.25395" width="0.4064" layer="16"/>
+<wire x1="52.07" y1="22.35905" x2="52.07" y2="24.13" width="0" layer="19" extent="1-16"/>
+<wire x1="60.96" y1="17.25395" x2="59.16395" y2="19.05" width="0.4064" layer="16"/>
+<wire x1="59.16395" y1="19.05" x2="54.90980625" y2="19.05" width="0.4064" layer="16"/>
 <wire x1="54.90980625" y1="19.05" x2="52.07" y2="21.88980625" width="0.4064" layer="16"/>
 <wire x1="52.07" y1="21.88980625" x2="52.07" y2="24.13" width="0.4064" layer="16"/>
-<wire x1="54.90980625" y1="19.05" x2="59.16395" y2="19.05" width="0.4064" layer="16"/>
-<wire x1="59.16395" y1="19.05" x2="62.97395" y2="15.24" width="0.4064" layer="16"/>
 </signal>
 <signal name="TX1_R">
@@
 <signal name="VCC">
 <contactref element="JP8" pad="9"/>
-<wire x1="78.74" y1="39.37" x2="82.55" y2="39.37" width="0.4064" layer="16"/>
-<contactref element="S1" pad="3.2"/>
-<wire x1="82.55" y1="39.37" x2="84.98" y2="41.8" width="0.4064" layer="16"/>
-<wire x1="84.98" y1="41.8" x2="84.98" y2="47.8" width="0.4064" layer="16"/>
 <contactref element="R4" pad="2"/>
 <contactref element="R3" pad="2"/>
 <wire x1="85.09" y1="36.83" x2="90.17" y2="36.83" width="0.4064" layer="16"/>
-<wire x1="85.09" y1="36.83" x2="82.55" y2="39.37" width="0.4064" layer="16"/>
+<contactref element="S3" pad="1"/>
+<wire x1="85.09" y1="36.83" x2="84.34605" y2="36.83" width="0.4064" layer="16"/>
+<wire x1="84.34605" y1="36.83" x2="81.80605" y2="39.37" width="0.4064" layer="16"/>
+<wire x1="81.80605" y1="39.37" x2="78.74" y2="39.37" width="0.4064" layer="16"/>
+<wire x1="87.63" y1="46.99" x2="87.63" y2="42.20980625" width="0.4064" layer="16"/>
+<wire x1="87.63" y1="42.20980625" x2="84.79019375" y2="39.37" width="0.4064" layer="16"/>
+<wire x1="84.79019375" y1="39.37" x2="78.74" y2="39.37" width="0.4064" layer="16"/>
 </signal>
 <signal name="GND2">
 <contactref element="JP8" pad="11"/>
-<contactref element="JP4" pad="1"/>
+<contactref element="BATT" pad="1"/>
 <wire x1="69.85" y1="45.72" x2="69.85" y2="44.45" width="0.4064" layer="16"/>
 <wire x1="69.85" y1="44.45" x2="71.12" y2="43.18" width="0.4064" layer="16"/>
@@
 </signal>
 <signal name="VCC2">
-<contactref element="JP4" pad="2"/>
-<contactref element="S1" pad="2.2"/>
-<wire x1="72.39" y1="45.72" x2="73.66" y2="45.72" width="0.4064" layer="16"/>
-<wire x1="73.66" y1="45.72" x2="74.93" y2="46.99" width="0.4064" layer="16"/>
-<wire x1="74.93" y1="46.99" x2="74.93" y2="49.53" width="0.4064" layer="16"/>
-<wire x1="74.93" y1="49.53" x2="76.2" y2="50.8" width="0.4064" layer="16"/>
-<wire x1="76.2" y1="50.8" x2="84.98" y2="50.8" width="0.4064" layer="16"/>
-<contactref element="JP5" pad="2"/>
+<contactref element="BATT" pad="2"/>
+<contactref element="ROUTER" pad="2"/>
 <wire x1="72.39" y1="45.72" x2="72.39" y2="46.69019375" width="0.4064" layer="16"/>
 <wire x1="72.39" y1="46.69019375" x2="69.55019375" y2="49.53" width="0.4064" layer="16"/>
@@
 <wire x1="58.94605" y1="49.53" x2="57.15" y2="47.73395" width="0.4064" layer="16"/>
 <wire x1="57.15" y1="47.73395" x2="57.15" y2="45.72" width="0.4064" layer="16"/>
+<contactref element="S3" pad="2"/>
+<wire x1="87.63" y1="49.53" x2="76.94395" y2="49.53" width="0.4064" layer="16"/>
+<wire x1="76.94395" y1="49.53" x2="74.93" y2="47.51605" width="0.4064" layer="16"/>
+<wire x1="74.93" y1="47.51605" x2="73.13395" y2="45.72" width="0.4064" layer="16"/>
+<wire x1="73.13395" y1="45.72" x2="72.39" y2="45.72" width="0.4064" layer="16"/>
 </signal>
 <signal name="N$3">
